File: PCBs/watch_main/fpga.kicad_sch (KiCad schematic)
At the start: 1 part, among them IC1201 ICE40UP5K-UWG30ITR1K

Commit message: PCB Schematic progress
Parts:
- added C1903 (x3), C1907: 4u7, Capacitor_SMD:C_0402_1005Metric, symbol Device:C_Small
- added C1904 (x3), C1911 (x3): 100n, Capacitor_SMD:C_0402_1005Metric, symbol Device:C_Small
- added R1201: 100R, Resistor_SMD:R_0402_1005Metric, symbol Device:R_Small
- added R1202: 10k, Resistor_SMD:R_0402_1005Metric, symbol Device:R_Small
- IC1201: footprint BGA30C40P5X6_211X254X60 -> watch_footprints:BGA30C40P5X6_211X254X60_modified
Connections:
- net +1V2: now also C1903.1, C1904.1, R1201.1; no longer IC1201.B2 (VCCPLL)
- net +1V8: now also C1907.1, C1911.1, C1911.1, C1911.1, R1202.1; no longer IC1201.B3 (IOT_46b_G0), IC1201.C3 (IOB_10a)
- net +3V3: now also C1903.1, C1904.1; no longer IC1201.D5 (IOB_2a)
- net CDONE: now also IC1201.E3 (IOB_13b); no longer IC1201.E4 (IOB_9b)
- net CRESET_B: now also R1202.2
- net CTRL: now also IC1201.F4 (IOB_11b_G5); no longer IC1201.A2 (IOT_37a)
- net GND: now also C1903.2, C1903.2, C1903.2, C1904.2, C1904.2, C1904.2, C1907.2, C1911.2, C1911.2, C1911.2
- net OLED_EN: now also IC1201.F2 (IOB_25b_G3); no longer IC1201.C5 (RGB2)
- net QSPI2.CS: now also IC1201.A5 (RGB0); no longer IC1201.B5 (RGB1)
- net QSPI2.IO1: now also IC1201.E5 (IOB_0a); no longer IC1201.F4 (IOB_11b_G5)
- net QSPI2.IO2: now also IC1201.D5 (IOB_2a); no longer IC1201.E5 (IOB_0a)
- net QSPI2.IO3: now also IC1201.E4 (IOB_9b); no longer IC1201.F2 (IOB_25b_G3)
- net QSPI2.SCK: now also IC1201.B5 (RGB1); no longer IC1201.A5 (RGB0)
- net INT renamed INT_NRF
- new net INT_STM: IC1201.A2 (IOT_37a)
- new net VCCPLL: C1903.1, C1904.1, IC1201.B2 (VCCPLL), R1201.2
- no-connect marks 1 -> 3
Other:
- note added: "VCC"
- note added: "VCCPLL"
- note added: "VDDIOx"
- note added: "VPP"
- note removed: "The following pins are used for routing and must be tri-stated: - IOB_2a - IOB_9b - IOB_10a - IOT_46b_G0"
- moved on the sheet: IC1201

Commit message: Started routing main PCB
Parts:
- R1201: renamed from R1202; now not fitted; now left out of the parts list
- renumbered R1201 to R1202
Other:
- note added: "CRESET_b must be pulled up by host"
- note added: "IOB_13b must be high-z"
- title: (none) -> Watch FPGA
