File: PCBs/watch_main/microphone.kicad_sch (KiCad schematic)
At the start: 2 parts

Commit message: Schematic finished and BOM started
Other:
- title: (none) -> Watch Microphone
Changed lines of the file:
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@@
 (kicad_sch (version 20230121) (generator eeschema)
   (paper "A4")
+  (title_block
+    (title "Watch Microphone")
+    (date "2023-12-20")
+    (rev "1")
+    (comment 1 "Checked by Ben Smith on 20/12/23")
+  )
   (junction (at 167.64 96.52) (diameter 0) (color 0 0 0 0)
   )
