File: PCBs/watch_main/stm32_power.kicad_sch (KiCad schematic)
At the start: 23 parts, among them U801 STM32U5A9NJH6Q

Commit message: Progress with schematic and RFID simulations
Parts:
- L1901: footprint (none) -> Inductor_SMD:L_0402_1005Metric
Changed lines of the file:
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@@
       (effects (font (size 1.27 1.27)) (justify left))
     )
-    (property "Footprint" "" (at 162.56 114.3 0)
+    (property "Footprint" "Inductor_SMD:L_0402_1005Metric" (at 162.56 114.3 0)
       (effects (font (size 1.27 1.27)) hide)
     )

Commit message: Schematic finished and BOM started
Parts:
- L1901: footprint Inductor_SMD:L_0402_1005Metric -> Inductor_SMD:L_Murata_DFE201610P
Changed lines of the file:
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@@
 (kicad_sch (version 20230121) (generator eeschema)
   (paper "A4")
+  (title_block
+    (rev "1")
+  )
   (junction (at 231.14 99.06) (diameter 0) (color 0 0 0 0)
   )
@@
       (effects (font (size 1.27 1.27)) (justify left))
     )
-    (property "Footprint" "Inductor_SMD:L_0402_1005Metric" (at 162.56 114.3 0)
-      (effects (font (size 1.27 1.27)) hide)
-    )
+    (property "Footprint" "Inductor_SMD:L_Murata_DFE201610P" (at 162.56 114.3 0)
+      (effects (font (size 1.27 1.27)) hide)
+    )

Commit message: Started routing main PCB
Parts:
- renumbered C1903 to C901, C1901 to C902, C1923 to C903, C1902 to C904, C1925 to C905, C1904 to C906, C1906 to C907, C1910 to C908, C1913 to C909, C1924 to C910, C1916 to C911, C1907 to C912, C1918 to C913, C1911 to C914, C1919 to C915, C1914 to C916, C1920 to C917, C1921 to C918, C1922 to C919, C1905 to C920, C1909 to C921, L1901 to L901
Other:
- title: (none) -> Watch Main MCU Power

Commit message: 69 Unrouted traces
Connections:
- net +3V3A is gone; now on net +3V3: C903.1, C905.1, U801.L6 (VDDA)
Changed lines of the file:
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@@
+    )
+  )
+  (symbol (lib_id "power:+3V3") (at 33.02 116.84 0) (unit 1)
+    (in_bom yes) (on_board yes) (dnp no) (fields_autoplaced)
+    (property "Reference" "#PWR0226" (at 33.02 120.65 0)
+      (effects (font (size 1.27 1.27)) hide)
+    )
+    (property "Value" "+3V3" (at 33.02 111.76 0)
+      (effects (font (size 1.27 1.27)))
+    )
+    (property "Footprint" "" (at 33.02 116.84 0)
+      (effects (font (size 1.27 1.27)) hide)
+    )
+    (property "Datasheet" "" (at 33.02 116.84 0)
+      (effects (font (size 1.27 1.27)) hide)
+    )
+    (pin "1")
+    (instances
+      (project "watch_main"
+        (path "/b008648a-c7cf-4e14-8a0a-b9314d757b4a/8f996a8c-7777-4a55-b361-37cede76953f"
+          (reference "#PWR0226") (unit 1)
+        )
+        (path "/b008648a-c7cf-4e14-8a0a-b9314d757b4a/8f147234-e39a-4c7c-8011-0af923cea553/79cbc0a6-b22c-4240-8664-408cf0e62ea6"
+          (reference "#PWR0905") (unit 1)
+        )
+      )
     )
   )
@@
     )
   )
-  (symbol (lib_id "watch_symbols_lib:+3V3A") (at 33.02 116.84 0) (unit 1)
-    (in_bom yes) (on_board yes) (dnp no) (fields_autoplaced)
-    (property "Reference" "#PWR0702" (at 33.02 120.65 0)
-      (effects (font (size 1.27 1.27)) hide)
-    )
-    (property "Value" "+3V3A" (at 33.02 111.76 0)
-      (effects (font (size 1.27 1.27)))
-    )
-    (property "Footprint" "" (at 33.02 116.84 0)
-      (effects (font (size 1.27 1.27)) hide)
-    )
-    (property "Datasheet" "" (at 33.02 116.84 0)
-      (effects (font (size 1.27 1.27)) hide)
-    )
-    (pin "1")
-    (instances
-      (project "watch_main"
-        (path "/b008648a-c7cf-4e14-8a0a-b9314d757b4a/8f147234-e39a-4c7c-8011-0af923cea553"
-          (reference "#PWR0702") (unit 1)
-        )
-        (path "/b008648a-c7cf-4e14-8a0a-b9314d757b4a/8f147234-e39a-4c7c-8011-0af923cea553/79cbc0a6-b22c-4240-8664-408cf0e62ea6"
-          (reference "#PWR0905") (unit 1)
-        )
-      )
-    )
-  )
   (symbol (lib_id "Device:C_Small") (at 71.12 88.9 0) (unit 1)
     (in_bom yes) (on_board yes) (dnp no)
@@
         (path "/b008648a-c7cf-4e14-8a0a-b9314d757b4a/8f147234-e39a-4c7c-8011-0af923cea553/79cbc0a6-b22c-4240-8664-408cf0e62ea6"
           (reference "#PWR0906") (unit 1)
+        )
+      )
+    )
+  )
+  (symbol (lib_id "power:+3V3") (at 157.48 127 0) (unit 1)
+    (in_bom yes) (on_board yes) (dnp no) (fields_autoplaced)
+    (property "Reference" "#PWR0226" (at 157.48 130.81 0)
+      (effects (font (size 1.27 1.27)) hide)
+    )
+    (property "Value" "+3V3" (at 157.48 121.92 0)
+      (effects (font (size 1.27 1.27)))
+    )
+    (property "Footprint" "" (at 157.48 127 0)
+      (effects (font (size 1.27 1.27)) hide)
+    )
+    (property "Datasheet" "" (at 157.48 127 0)
+      (effects (font (size 1.27 1.27)) hide)
+    )
+    (pin "1")
+    (instances
+      (project "watch_main"
+        (path "/b008648a-c7cf-4e14-8a0a-b9314d757b4a/8f996a8c-7777-4a55-b361-37cede76953f"
+          (reference "#PWR0226") (unit 1)
+        )
+        (path "/b008648a-c7cf-4e14-8a0a-b9314d757b4a/8f147234-e39a-4c7c-8011-0af923cea553/79cbc0a6-b22c-4240-8664-408cf0e62ea6"
+          (reference "#PWR0911") (unit 1)
         )
       )
@@
         )
       )
-    )
-  )
-  (symbol (lib_id "watch_symbols_lib:+3V3A") (at 157.48 127 0) (unit 1)
-    (in_bom yes) (on_board yes) (dnp no) (fields_autoplaced)
-    (property "Reference" "#PWR0702" (at 157.48 130.81 0)
-      (effects (font (size 1.27 1.27)) hide)
-    )
-    (property "Value" "+3V3A" (at 157.48 121.92 0)
-      (effects (font (size 1.27 1.27)))
-    )
-    (property "Footprint" "" (at 157.48 127 0)
-      (effects (font (size 1.27 1.27)) hide)
-    )
-    (property "Datasheet" "" (at 157.48 127 0)
-      (effects (font (size 1.27 1.27)) hide)
-    )
-    (pin "1")
-    (instances
-      (project "watch_main"
-        (path "/b008648a-c7cf-4e14-8a0a-b9314d757b4a/8f147234-e39a-4c7c-8011-0af923cea553"
-          (reference "#PWR0702") (unit 1)
-        )
-        (path "/b008648a-c7cf-4e14-8a0a-b9314d757b4a/8f147234-e39a-4c7c-8011-0af923cea553/79cbc0a6-b22c-4240-8664-408cf0e62ea6"
-          (reference "#PWR0911") (unit 1)
-        )
-      )

Commit message: Test rig board finished
Other:
- note added: "VDDIO2 is 3V3 to interface with touch sensor"
- note removed: "VDDIO2 is 3V3 to interface with GNSS module"
Changed lines of the file:
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@@
     (fill (type none))
   )
-  (text "VDDIO2 is 3V3 to interface\nwith GNSS module" (at 93.98 66.04 0)
+  (text "VDDIO2 is 3V3 to interface\nwith touch sensor" (at 93.98 66.04 0)
     (effects (font (size 1.27 1.27)) (justify left bottom))
   )
