File: PCBs/watch_test_rig/watch_test_rig.kicad_pcb (KiCad board)
At the start: 2 copper layers, 19 parts, among them J101 STDC14, J102 MIPI10

Commit message: Started routing main PCB
Parts:
- removed PP117: 8mm, watch_footprints:Pogo_Pin_8mm
- added D101: GREEN, Diode_SMD:D_0603_1608Metric, F.Cu at (141.6, 76.3)
- added D102: GREEN, Diode_SMD:D_0603_1608Metric, F.Cu at (141.6, 78.9)
- added D103: GREEN, Diode_SMD:D_0603_1608Metric, F.Cu at (141.6, 81.4)
- added D104: GREEN, Diode_SMD:D_0603_1608Metric, F.Cu at (141.6, 84.0)
- added D105: GREEN, Diode_SMD:D_0603_1608Metric, F.Cu at (141.6, 86.6)
- added J103: HRO_TYPE-C-31-M-12, watch_footprints:TYPE-C-31-M-12, F.Cu at (145.6, 71.6)
- added PP118: 8mm, watch_footprints:Pogo_Pin_8mm, F.Cu at (137.6, 82.9)
- added PP119: 8mm, watch_footprints:Pogo_Pin_8mm, F.Cu at (137.6, 86.9)
- added Q101: DMN21D2UFB-7B, watch_footprints:DMN21D2UFB7B, F.Cu at (156.7, 66.1)
- added Q102: DMN21D2UFB-7B, watch_footprints:DMN21D2UFB7B, F.Cu at (156.7, 68.6)
- added Q103: DMN21D2UFB-7B, watch_footprints:DMN21D2UFB7B, F.Cu at (156.7, 71.0)
- added Q104: DMN21D2UFB-7B, watch_footprints:DMN21D2UFB7B, F.Cu at (156.7, 73.5)
- added R101: 2k2, Resistor_SMD:R_0402_1005Metric, F.Cu at (154.7, 76.0)
- added R102: 2k2, Resistor_SMD:R_0402_1005Metric, F.Cu at (154.7, 78.0)
- added R103: 2k2, Resistor_SMD:R_0402_1005Metric, F.Cu at (154.7, 79.9)
- added R104: 2k2, Resistor_SMD:R_0402_1005Metric, F.Cu at (154.7, 81.9)
- added R105: 2k2, Resistor_SMD:R_0402_1005Metric, F.Cu at (154.7, 83.9)
- moved PP105 23.8 mm to (129.6, 82.9)
- moved PP106 23.8 mm to (129.6, 86.9)
- moved PP107 22.6 mm to (133.6, 66.9)
- moved PP101 21.3 mm to (129.6, 66.9)
- moved PP102 21.3 mm to (129.6, 70.9)
- moved PP103 21.3 mm to (129.6, 74.9)
- moved PP104 21.3 mm to (129.6, 78.9)
- moved PP113 20.6 mm to (137.6, 66.9)
- moved J101 20.1 mm to (148.5, 80.4)
- moved J102 20.1 mm to (148.5, 90.1)
- moved PP114 15.2 mm to (137.6, 70.9)
- moved PP115 15.2 mm to (137.6, 74.9)
- moved PP116 14.1 mm to (137.6, 78.9)
- moved PP112 10.5 mm to (133.6, 86.9)
- moved PP108 9.99 mm to (133.6, 70.9)
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Connections:
- PP110 pad 1: +1V8 -> VBUS
- PP111 pad 1: GND -> +VBAT
- PP114 pad 1: +1V2 -> GND
- PP116 pad 1: +VBAT -> /LED_STM32

Commit message: Main PCB placement and routing progress
Parts:
- moved PP107 1.22 mm to (134.8, 66.9)

Commit message: Main PCB finished
Parts:
- added C101: 100n, Capacitor_SMD:C_0402_1005Metric, F.Cu at (83.2, 109.6)
- added C102: 100n, Capacitor_SMD:C_0402_1005Metric, F.Cu at (83.2, 111.6)
- added H101: M3, MountingHole:MountingHole_3.2mm_M3_DIN965_Pad_TopBottom, F.Cu at (212.0, 58.0)
- added H102: M3, MountingHole:MountingHole_3.2mm_M3_DIN965_Pad_TopBottom, F.Cu at (212.0, 132.0)
- added H103: M3, MountingHole:MountingHole_3.2mm_M3_DIN965_Pad_TopBottom, F.Cu at (118.0, 132.0)
- added H104: M3, MountingHole:MountingHole_3.2mm_M3_DIN965_Pad_TopBottom, F.Cu at (118.0, 58.0)
- added H105: M3, MountingHole:MountingHole_3.2mm_M3_DIN965_Pad_TopBottom, F.Cu at (154.5, 71.5)
- added H106: M3, MountingHole:MountingHole_3.2mm_M3_DIN965_Pad_TopBottom, F.Cu at (198.5, 71.5)
- added H107: M3, MountingHole:MountingHole_3.2mm_M3_DIN965_Pad_TopBottom, F.Cu at (154.5, 118.5)
- added H108: M3, MountingHole:MountingHole_3.2mm_M3_DIN965_Pad_TopBottom, F.Cu at (198.5, 118.5)
- added J105: Conn_02x03_Odd_Even, Connector_PinHeader_2.54mm:PinHeader_2x03_P2.54mm_Vertical, F.Cu at (185.6, 125.8)
- added PP117: 8mm, watch_footprints:Pogo_Pin_8mm, F.Cu at (177.9, 113.0)
- added PP120: 8mm, watch_footprints:Pogo_Pin_8mm, F.Cu at (185.7, 110.2)
- added PP121: 8mm, watch_footprints:Pogo_Pin_8mm, F.Cu at (188.2, 107.8)
- added PP122: 8mm, watch_footprints:Pogo_Pin_8mm, F.Cu at (181.3, 112.8)
- added R106: 5k1, Resistor_SMD:R_0402_1005Metric, F.Cu at (87.3, 82.8)
- added R107: 5k1, Resistor_SMD:R_0402_1005Metric, F.Cu at (87.3, 84.8)
- added SW101: PSH_BTN, Button_Switch_THT:SW_PUSH_6mm_H5mm, F.Cu at (140.1, 130.2)
- added SW102: PSH_BTN, Button_Switch_THT:SW_PUSH_6mm_H5mm, F.Cu at (127.8, 130.2)
- added SW103: SW_SPDT, Connector_PinHeader_2.54mm:PinHeader_1x03_P2.54mm_Vertical, F.Cu at (139.5, 62.0)
- added TP101: 2mm, TestPoint:TestPoint_Pad_D2.0mm, F.Cu at (168.0, 61.0)
- added TP102: 2mm, TestPoint:TestPoint_Pad_D2.0mm, F.Cu at (161.0, 61.0)
- added TP103: 2mm, TestPoint:TestPoint_Pad_D2.0mm, F.Cu at (175.0, 61.0)
- added TP104: 2mm, TestPoint:TestPoint_Pad_D2.0mm, F.Cu at (196.0, 61.0)
- added TP105: 2mm, TestPoint:TestPoint_Pad_D2.0mm, F.Cu at (189.0, 61.0)
- added TP106: 2mm, TestPoint:TestPoint_Pad_D2.0mm, F.Cu at (182.0, 61.0)
- added U101: Watch_Outline, watch_footprints:Watch Outline V1, F.Cu at (175.7, 95.2)
- J103: value HRO_TYPE-C-31-M-12 -> TYPE-C-31-M-12
- moved Q101 77.7 mm to (85.2, 96.6)
- moved Q102 77.7 mm to (85.2, 99.0)
- moved Q103 77.7 mm to (85.2, 101.5)
- moved Q104 77.7 mm to (85.2, 104.0)
- moved R101 54.0 mm to (102.2, 63.4)
- moved R102 54.0 mm to (102.2, 65.4)
- moved R103 54.0 mm to (102.2, 67.4)
- moved R104 54.0 mm to (102.2, 69.4)
- moved R105 54.0 mm to (102.2, 71.4)
- moved PP110 52.4 mm to (185.9, 77.0)
- moved PP105 50.4 mm to (179.0, 92.9)
- moved PP116 50.3 mm to (187.1, 87.5)
- moved PP104 50.2 mm to (179.5, 84.2)
- moved PP107 50.1 mm to (176.2, 95.1)
- moved PP112 50.0 mm to (183.0, 79.3)
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Connections:
- net Net-(J103-VBUS-PadA4_B9) renamed /VIN
- J103 pad A1_B12: Net-(J103-GND-PadA1_B12) -> GND
- J103 pad A5: unconnected-(J103-CC1-PadA5) -> /CC1
- J103 pad B1_A12: Net-(J103-GND-PadA1_B12) -> GND
- J103 pad B5: unconnected-(J103-CC2-PadB5) -> /CC2
Routing:
- added copper zone on B.Cu, net GND
Other:
- board outline added: 100 x 80 mm

Commit message: Test rig board finished
Parts:
- removed TP101, TP102, TP103, TP104, TP105, TP106: 2mm, TestPoint:TestPoint_Pad_D2.0mm
- added J106: Conn_02x05_Odd_Even, Connector_PinHeader_2.54mm:PinHeader_2x05_P2.54mm_Vertical, F.Cu at (171.4, 64.3)
- U101: value Watch_Outline -> Watch_Outline SS; footprint watch_footprints:Watch Outline V1 -> watch_footprints:Watch Outline V1 SS
- moved Q104 70.6 mm to (146.5, 69.0), turned to 90 degrees
- moved Q103 65.9 mm to (142.5, 69.0), turned to 90 degrees
- moved Q102 61.2 mm to (138.5, 69.0), turned to 90 degrees
- moved C101 60.1 mm to (142.5, 119.5), turned to 180 degrees
- moved Q101 56.5 mm to (134.5, 69.0), turned to 90 degrees
- moved C102 47.5 mm to (130.0, 119.5), turned to 180 degrees
- moved R105 44.3 mm to (146.5, 72.5), turned to 90 degrees
- moved R107 41.4 mm to (125.4, 68.5), turned to -90 degrees
- moved D104 41.4 mm to (130.5, 76.5), turned to -90 degrees
- moved R103 40.6 mm to (142.5, 72.5), turned to 90 degrees
- moved R106 39.6 mm to (125.4, 72.0), turned to 90 degrees
- moved R102 37.0 mm to (138.5, 72.5), turned to 90 degrees
- moved R101 33.5 mm to (134.5, 72.5), turned to 90 degrees
- moved D103 28.7 mm to (142.5, 76.5), turned to -90 degrees
- moved R104 28.5 mm to (130.5, 72.5), turned to 90 degrees
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Connections:
- D101 pad 2: /LED_3V3_A -> VBUS
- D102 pad 2: /LED_1V8_A -> VBUS
- D103 pad 2: /LED_1V2_A -> VBUS
- D104 pad 1: GND -> /LED_VBUS_K
- D104 pad 2: /LED_VBUS_A -> VBUS
- D105 pad 2: /LED_STM32_A -> VBUS
- Q101 pad 3: /LED_3V3_K -> /LED_3V3_D
- Q102 pad 3: /LED_1V8_K -> /LED_1V8_D
- Q103 pad 3: /LED_1V2_K -> /LED_1V2_D
- Q104 pad 3: /LED_STM32_K -> /LED_STM32_D
- R101 pad 1: VBUS -> /LED_3V3_K
- R101 pad 2: /LED_3V3_A -> /LED_3V3_D
- R102 pad 1: VBUS -> /LED_1V8_K
- R102 pad 2: /LED_1V8_A -> /LED_1V8_D
- R103 pad 1: VBUS -> /LED_1V2_K
- R103 pad 2: /LED_1V2_A -> /LED_1V2_D
- R104 pad 1: VBUS -> /LED_VBUS_K
- R104 pad 2: /LED_VBUS_A -> GND
- R105 pad 1: VBUS -> /LED_STM32_K
- R105 pad 2: /LED_STM32_A -> /LED_STM32_D
Routing:
- net +1V8: track 0.00 -> 130.7 mm, vias 0 -> 2
- net /STM32_RST: track 0.00 -> 104.7 mm
- net /NRF_RST: track 0.00 -> 100.5 mm
- net /STM32_VCP_TX: track 0.00 -> 85.5 mm
- net /STM32_VCP_RX: track 0.00 -> 72.9 mm
- net +3V3: track 0.00 -> 71.7 mm
- net /STM32_SWO: track 0.00 -> 52.7 mm
- net /LED_STM32: track 0.00 -> 52.3 mm, vias 0 -> 2
- net +1V2: track 0.00 -> 47.6 mm
- net /STM32_SWDIO: track 0.00 -> 41.7 mm
- net /STM32_SWCLK: track 0.00 -> 40.9 mm
- net /NRF_SWDIO: track 0.00 -> 33.4 mm
- net /NRF_SWCLK: track 0.00 -> 32.1 mm
- net GND: track 0.00 -> 28.2 mm, vias 0 -> 16
- net /RF: track 0.00 -> 24.7 mm
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- added copper zone on F.Cu, net /VIN
- added copper zone on F.Cu, net VBUS
Other:
- outline, holes or cut-outs redrawn
- board text added: "1"
- board text added: "10"
- board text added: "13"
- board text added: "14"
- board text added: "1V2"
- board text added: "1V8"
- board text added: "2"
- board text added: "3V3"
- board text added: "9"
- board text added: "Designed by Ben Smith 2023"
- board text added: "ENV"
- board text added: "GND"
- board text added: "GPIO"
- board text added: "NRF53 DEBUG"
- board text added: "NRF53 RESET"
- board text added: "OFF"
- board text added: "ON"
- board text added: "RF"
- board text added: "RF_IN"
- board text added: "STM32 DEBUG"
- board text added: "STM32 RESET"
- board text added: "VBAT"
- board text added: "VBUS"
- board text added: "Watch Test Rig v1"
