File: PCBs/watch_test_rig v2/watch_test_rig.kicad_sch (KiCad schematic)
At the start: 54 parts, among them J101 STDC14, J102 MIPI10, J103 TYPE-C-31-M-12, J104 Conn_02x04_Odd_Even, Q101 DMN21D2UFB-7B, Q102 DMN21D2UFB-7B, Q103 DMN21D2UFB-7B, Q104 DMN21D2UFB-7B, SW101 SW_SPDT, SW102 PSH_BTN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

Commit message: Main board and test rig complete & ordered.
Parts:
- removed H101, H102, H103, H104: M3, MountingHole:MountingHole_3.2mm_M3_DIN965_Pad_TopBottom, symbol Mechanical:MountingHole_Pad
- removed U101: Watch_Outline_V2_SS, watch_footprints:Watch Outline V2 SS, symbol watch_symbols_lib:Watch_Outline_V2_SS
- added D106: GREEN, Diode_SMD:D_0603_1608Metric, symbol Device:LED_Small
- added J106: Conn_02x03_Odd_Even, Connector_PinHeader_2.54mm:PinHeader_2x03_P2.54mm_Vertical, symbol Connector_Generic:Conn_02x03_Odd_Even
- added PP121, PP122: 8mm, watch_footprints:Pogo_Pin_8mm_SMD, symbol watch_symbols_lib:Pogo_Pin_8mm_SMD
- added Q105: DMN21D2UFB-7B, watch_footprints:DMN21D2UFB7B, symbol DMN21D2UFB-7B:DMN21D2UFB-7B
- added R108: 2k2, Resistor_SMD:R_0402_1005Metric, symbol Device:R_Small
- added U101: Watch_Outline_V2_SS_Inverted, watch_footprints:Watch Outline V2 SS Inverted, symbol watch_symbols_lib:Watch_Outline_V2_SS_Inverted
- PP101, PP102, PP103, PP104, PP105, PP106, PP107, PP108, PP109, PP110, PP111, PP112, PP113, PP114, PP115, PP116, PP117, PP118, PP119, PP120: footprint TestPoint:TestPoint_Pad_D2.0mm -> watch_footprints:Pogo_Pin_8mm_SMD
Connections:
- net +1V8: now also J104.4 (Pin_4); no longer J104.2 (Pin_2)
- net +3V3: now also J104.6 (Pin_6); no longer J104.4 (Pin_4)
- net +VBAT: now also J104.2 (Pin_2); no longer J104.6 (Pin_6)
- net GND: now also J106.1 (Pin_1), J106.3 (Pin_3), J106.5 (Pin_5), PP121.1, Q105.2 (S)
- net GPIO1: now also J106.2 (Pin_2)
- net GPIO2: now also J106.4 (Pin_4)
- net VBUS: now also D106.2 (A)
- net GPIO2_D_K renamed GPIO2_K
- new net GPIO3: J106.6 (Pin_6), PP122.1, Q105.1 (G)
- new net GPIO3_D: Q105.3 (D), R108.2
- new net GPIO3_K: D106.1 (K), R108.1
Other:
- note added: "Power + GPIO Headers"
- note removed: "Power Header"
- moved on the sheet: D101, D102, D103, D104, D105, H105, H106, H107, H108, J104, PP112, PP113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
