File: PCBs/watch_main_v3/bluetooth.kicad_sch (KiCad schematic)
At the start: 24 parts, among them U301 NRF5340-QKAA-R7, Y301 32MHz

Commit message: Started watch_main_v3
Parts:
- removed C301, C302, C310, C311, C316: 1u, Capacitor_SMD:C_0402_1005Metric, symbol Device:C_Small
- removed C303, C304, C305, C306, C308, C309, C312, C313, C314: 100n, Capacitor_SMD:C_0402_1005Metric, symbol Device:C_Small
- removed C307: 2n2, Capacitor_SMD:C_0402_1005Metric, symbol Device:C_Small
- removed C315: 0p7, Capacitor_SMD:C_0402_1005Metric, symbol Device:C_Small
- removed L301, L302: 10u, Inductor_SMD:L_TDK_MLZ1608, symbol Device:L_Small
- removed L303: 2n2, Inductor_SMD:L_0402_1005Metric, symbol Device:L_Small
- removed TP804, TP805 (x2): 1.5mm, TestPoint:TestPoint_Pad_D1.5mm, symbol Connector:TestPoint_Small
- removed U301: NRF5340-QKAA-R7, watch_footprints:NRF5340-QKAA-R7_modified, symbol NRF5340-QKAA-R7:NRF5340-QKAA-R7
- removed Y301: 32MHz, Crystal:Crystal_SMD_2016-4Pin_2.0x1.6mm, symbol Device:Crystal_GND24_Small
Connections:
- no-connect marks 61 -> 0
Other:
- note removed: "50mA Inductors"
- note removed: "NP0 Cap"
- note removed: "nRF5340 Product specification p798"
