File: PCBs/watch_main_v3/antenna.kicad_sch (KiCad schematic)
At the start: 9 parts, among them U1601 GPS_&_BT_Antenna_Keepout

Commit message: PCB V3 progress
Connections:
- net RF_2.4G renamed RF_2.4G/5G
