File: PCBs/watch_main_v3/stm32.kicad_sch (KiCad schematic)
At the start: 21 parts, among them Y801 16MHz, Y802 32.768kHz

Commit message: watch_main_v3 WiFi/Bluetooth schematic done
Parts:
- added R811, R812: 4k7, Resistor_SMD:R_0402_1005Metric, symbol Device:R_Small
Connections:
- net I2C6.SCL: now also R811.2; no longer R809.2
- net I2C6.SDA: now also R812.2; no longer R810.2
- removed net +1V8: R801.1, R802.1, R803.1, R804.1, R805.1, R806.1, R809.1, R810.1
- net +3V3: no longer names the net of R807.1, R808.1
- new net: R805.1, R806.1
- new net: R803.1, R804.1
- new net: R811.1, R812.1
- new net: R801.1, R802.1
- new net: R809.1, R810.1
- new net I2C5.SCL: R809.2
- new net I2C5.SDA: R810.2
- no-connect marks 75 -> 0
Other:
- moved on the sheet: C801, C802, C803, C804, R801, R802, R803, R804, R805, R806, R807, R808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

Commit message: PCB V3 progress
Parts:
- removed TP804: 1.5mm, TestPoint:TestPoint_Pad_D1.5mm, symbol Connector:TestPoint_Small
- added U801: STM32U5G9ZJJ6Q, watch_footprints:UFBGA144_STM, symbol STM32U5G9ZJJ6Q:STM32U5G9ZJJ6Q
- renumbered R805 to R801, R807 to R802, R806 to R803, R808 to R804, R809 to R805, R801 to R806, R810 to R807, R802 to R808, R811 to R809, R803 to R810, R812 to R811, R804 to R812, TP805 to TP801, TP806 to TP802, TP807 to TP803, TP801 to TP804
Connections:
- net ADF1_CCK0: now also U801.K6 (PE9)
- net ADF1_SDI0: now also U801.J7 (PE10)
- net ALS_INT: now also U801.J6 (PG1)
- net AVDDEN: now also U801.D3 (PE6)
- net BTN: now also U801.M9 (PB15)
- net DISPLAY_RST: now also U801.A3 (PH3_BOOT0)
- net DSI.CKN: now also U801.F1 (DSI_CKN)
- net DSI.CKP: now also U801.F2 (DSI_CKP)
- net DSI.D0N: now also U801.E1 (DSI_D0N)
- net DSI.D0P: now also U801.E2 (DSI_D0P)
- net DSI_TE: now also U801.C5 (PB7)
- net FLASH_INT: now also U801.G9 (PC6)
- net FLASH_RST: now also U801.H12 (PH13)
- net FLASH_RSTO: now also U801.F9 (PC7)
- net GNSS_RST: now also U801.B6 (PG15)
- net GNSS_WAKEUP: now also U801.A6 (PG14)
- net GPIO1: now also U801.G5 (PC2)
- net GPIO2: now also U801.G4 (PF2)
- net GPIO3: now also U801.C6 (PG13)
- net HR_INT: now also U801.L11 (PD10)
- net I2C1.SCL: now also U801.A4 (PB6)
- net I2C1.SDA: now also U801.A2 (PB9)
- net I2C2.SCL: now also U801.M10 (PB13)
- net I2C2.SDA: now also U801.L7 (PB11)
- net I2C3.SCL: now also U801.K2 (PC0)
- net I2C3.SDA: now also U801.K1 (PC1)
- net I2C4.SCL: now also U801.K11 (PD12)
- net I2C4.SDA: now also U801.K9 (PD13)
- net I2C5.SCL: now also U801.E7 (PD1)
- net I2C5.SDA: now also U801.D8 (PD0)
- net I2C6.SCL: now also U801.F4 (PF1)
- net I2C6.SDA: now also U801.E5 (PF0)
- net IMU_INT1: now also U801.C4 (PE5)
- net IMU_INT2: now also U801.E4 (PC13)
- net LRA_EN: now also U801.L12 (PD14)
- net MAG_INT: now also U801.H8 (PE8)
- net OSC32_IN: now also U801.C1 (PC14-OSC32_IN)
- net OSC32_OUT: now also U801.D2 (PC15-OSC32_OUT)
- net OSC_IN: now also U801.H2 (PH0-OSC_IN)
- net OSC_OUT: now also U801.J1 (PH1-OSC_OUT)
- net OSPI1.CLKN: now also U801.B5 (PB5)
- net OSPI1.CLKP: now also U801.K8 (PB10)
- net OSPI1.CS: now also U801.M5 (PE11)
- net OSPI1.DQS: now also U801.H6 (PB2)
- net OSPI1.IO0: now also U801.J8 (PE12)
- net OSPI1.IO1: now also U801.L6 (PE13)
- net OSPI1.IO2: now also U801.K7 (PE14)
- net OSPI1.IO3: now also U801.M6 (PE15)
- net OSPI1.IO4: now also U801.K12 (PH9)
- net OSPI1.IO5: now also U801.J12 (PH10)
- net OSPI1.IO6: now also U801.J11 (PH11)
- net OSPI1.IO7: now also U801.H11 (PH12)
- net PWR_ENCHG: now also U801.M11 (PD8)
- net PWR_INT: now also U801.K10 (PD9)
- net SDMMC1.CK: now also U801.A11 (PC12)
- net SDMMC1.CKIN: now also U801.B4 (PB8)
- net SDMMC1.CMD: now also U801.B9 (PD2)
- net SDMMC1.D0: now also U801.D12 (PC8)
- net SDMMC1.D1: now also U801.F8 (PC9)
- net SDMMC1.D2: now also U801.B10 (PC10)
- net SDMMC1.D3: now also U801.C8 (PC11)
- net SDMMC2.CK: now also U801.D7 (PD6)
- net SDMMC2.CMD: now also U801.A9 (PD7)
- net SDMMC2.D0: now also U801.L10 (PB14)
- net SDMMC2.D1: now also U801.D11 (PA8)
- net SDMMC2.D2: now also U801.D6 (PB3)
- net SDMMC2.D3: now also U801.A5 (PB4)
- net SD_CD: now also U801.K5 (PG0)
- net SD_EN: now also U801.L5 (PE7)
- net SPI1.CS: now also U801.J5 (PB0)
- net SPI1.MISO: now also U801.M3 (PA6)
- net SPI1.MOSI: now also U801.L4 (PA7)
- net SPI1.SCK: now also U801.K4 (PA5)
- net SWD.RST: now also U801.J2 (NRST)
- net SWD.SWCLK: now also U801.B11 (PA14)
- net SWD.SWDIO: now also U801.C10 (PA13)
- net SWIRE_IN: now also U801.B3 (PE0)
- net SWIRE_OUT: now also U801.C3 (PE4)
- net TOUCH_INT: now also U801.L9 (PD11)
- net TOUCH_RST: now also U801.H9 (PD15)
- net TP_INT: now also U801.B1 (PE2)
- net TP_RST: now also U801.B2 (PE3)
- net USART1.RX: now also U801.A8 (PG10)
- net USART1.TX: now also U801.B7 (PG9)
- net USB.DN: now also U801.C12 (PA11)
- net USB.DP: now also U801.C11 (PA12)
- net +1V8: now reaches R801.1, R803.1
- net +1V8: now also R802.1, R804.1, R805.1, R806.1, R807.1, R808.1, R810.1, R812.1
- net +3V3: now reaches R809.1, R811.1
- new net AVDD_ADC: U801.M2 (PA3)
- new net BT_DEV_WAKE: U801.E11 (PI2)
- new net BT_EN: U801.F11 (PI0)
- new net BT_HOST_WAKE: U801.E12 (PI3)
- new net ELVDD_ADC: U801.L3 (PA4)
- new net ELVSS_ADC: U801.L1 (PC3)
- new net GNSS_PPS: U801.A7 (PG12)
- new net RCC_LSCO: U801.L2 (PA2)
- new net UART4.RX: U801.K3 (PA1)
- new net UART4.TX: U801.H4 (PA0)
- new net USART2.CTS: U801.A10 (PD3)
- new net USART2.RTS: U801.C7 (PD4)
- new net USART2.RX: U801.C9 (PA15)
- new net USART2.TX: U801.B8 (PD5)
- new net VBUS_ADC: U801.M4 (PB1)
- new net WL_BT_PWR_EN: U801.G12 (PH15)
- new net WL_EN: U801.F12 (PI1)
- new net WL_HOST_WAKE: U801.G11 (PH14)
- no-connect marks 0 -> 4
Other:
- moved on the sheet: TP801, TP802, TP803, TP804
