File: PCBs/watch_main_v3/power.kicad_sch (KiCad schematic)
At the start: 18 parts, among them IC201 ADP5360ACBZ-2-R7, Q201 DMP2104LP-7

Commit message: PCB V3 progress
Parts:
- renumbered TP802 to TP201, TP802 to TP202, TP802 to TP203, TP802 to TP204

Commit message: PCB V3 Progress
Parts:
- added R203: 50m, Resistor_SMD:R_0402_1005Metric, symbol Device:R_Small
- added U201: MAX9938TEBS+TG45, watch_footprints:BGA4C50P2X2_100X100X67, symbol MAX9938TEBS+TG45:MAX9938TEBS+TG45
Connections:
- net +VSYS: now also R203.2, U201.A2 (RS-); no longer C204.1, IC201.E6 (VSYS)
- net GND: now also U201.B1 (GND)
- new net ISYS: U201.B2 (OUT)
- new net VSYS_MON: C204.1, IC201.E6 (VSYS), R203.1, U201.A1 (RS+)
Other:
- note added: "73uA Per LSB"
- moved on the sheet: C204

Commit message: Hard routing done
Parts:
- added D201: LED_R, LED_SMD:LED_0402_1005Metric, symbol Device:LED_Small
- added D202: LED_G, LED_SMD:LED_0402_1005Metric, symbol Device:LED_Small
- added D203: LED_B, LED_SMD:LED_0402_1005Metric, symbol Device:LED_Small
- added R204, R205, R206: 1k, Resistor_SMD:R_0402_1005Metric, symbol Device:R_Small
- added TP205: 1.5mm, TestPoint:TestPoint_Pad_D1.5mm, symbol Connector:TestPoint_Small
- added U202: PCA9570GMH, watch_footprints:PCA9570GMH, symbol PCA9570GMH:PCA9570GMH
Connections:
- net +1V8: now also R204.1, R205.1, R206.1, U202.8 (VDD)
- net +VSYS: now also TP205.1
- net GND: now also U202.4 (VSS)
- net I2C.SCL: now also U202.6 (SCL)
- net I2C.SDA: now also U202.7 (SDA)
- new net LED_B_A: D203.2 (A), R206.2
- new net LED_B_K: D203.1 (K), U202.3 (P2)
- new net LED_G_A: D202.2 (A), R205.2
- new net LED_G_K: D202.1 (K), U202.2 (P1)
- new net LED_R_A: D201.2 (A), R204.2
- new net LED_R_K: D201.1 (K), U202.1 (P0)
- no-connect marks 6 -> 7
Other:
- moved on the sheet: C201, C202, C203, C204, C205, C206, C207, C208, IC201, L201, L202, Q201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
