File: PCBs/watch_main_v3/wifi_bluetooth.kicad_sch (KiCad schematic)
At the start: 17 parts, among them IC1102 LQ05041QCS6, U301 LBEE5PK2AE_564

Commit message: PCB V3 progress
Parts:
- renumbered C1101 to C301, C1101 to C302, C1101 to C303, C1101 to C304, C1101 to C305, IC1102 to IC301, IC1102 to IC302, L1404 to L301, R401 to R301, R401 to R302, R401 to R303, R401 to R304, R401 to R305, TP802 to TP301, TP803 to TP302, TP803 to TP303
Connections:
- net WL_BT_EN renamed WL_BT_PWR_EN
Other:
- moved on the sheet: C301, C302, C303, C304, C305, IC301, IC302, L301, U301B

Commit message: DISPLAY WORKS!!!
Other:
- note added: "Setting EN high turns on wireless"
Changed lines of the file:
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@@
+		)
+	)
+	(text "Setting EN high\nturns on wireless"
+		(exclude_from_sim no)
+		(at 30.48 152.4 0)
+		(effects
+			(font
+				(size 1.27 1.27)
+			)
 		)
 	)
