File: PCBs/rfid_module_v1.1/boost_converter.kicad_sch (KiCad schematic)
At the start: 8 parts, among them IC501 MAX17291BANT+T

Commit message: Added comments to RFID module and created gerber files.
Other:
- note added: "Boost converter to change RFID transmission power."
- note added: "FB_OFFSET varying from 0 to 3v3 changes VRF from 16V to 5V5."
Changed lines of the file:
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@@
     (stroke (width 0) (type default))
+  )
+  (text "Boost converter to change RFID transmission power.\n"
+    (at 116.84 134.62 0)
+    (effects (font (size 1.27 1.27)) (justify left bottom))
+  )
+  (text "FB_OFFSET varying from 0 to 3v3\nchanges VRF from 16V to 5V5."
+    (at 172.72 106.68 0)
+    (effects (font (size 1.27 1.27)) (justify left bottom))
   )
   (label "FB" (at 160.02 96.52 0) (fields_autoplaced)
