File: PCBs/rfid_module_v1.1/pogo_connector.kicad_sch (KiCad schematic)
At the start: 4 parts, among them J401 10-Pin_Pogo_Connector_Male, Q203 DMN21D2UFB-7B

Commit message: PCB V3 progress
Parts:
- renumbered Q203 to Q401
