File: PCBs/rfid_module_v1.1/rfid.kicad_sch (KiCad schematic)
At the start: 47 parts, among them IC201 TLV9004SIRTER, IC202 MAX9027EBT+T, Q201 DMN21D2UFB-7B, Q202 DMP21D5UFB4-7B, Q203 DMN21D2UFB-7B, Q204 DMN21D2UFB-7B

Commit message: Minor PCB fixes
Parts:
- Q202: value DMP21D5UFB4-7B -> BSS84AKM,315; Mouser Part Number 621-DMP21D5UFB4-7B -> 771-BSS84AKM315; Mouser Price/Stock https://www.mouser.co.uk/ProductDetail/Diodes-Incorporated/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 -> https://www.mouser.co.uk/ProductDetail/Nexperia/BSS84AKM315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
Changed lines of the file:
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@@
       (effects (font (size 1.27 1.27)) (justify left))
     )
-    (property "Value" "DMP21D5UFB4-7B" (at 81.28 35.56 0)
+    (property "Value" "BSS84AKM,315 " (at 81.28 35.56 0)
       (effects (font (size 1.27 1.27)) (justify left))
     )
@@
       (effects (font (size 1.27 1.27)) (justify left top) hide)
     )
-    (property "Datasheet" "https://componentsearchengine.com/Datasheets/1/DMP21D5UFB4-7B.pdf" (at 82.55 -158.09 0)
+    (property "Datasheet" "https://www.mouser.co.uk/datasheet/2/916/BSS84AKM-1509379.pdf" (at 82.55 -158.09 0)
       (effects (font (size 1.27 1.27)) (justify left top) hide)
     )
@@
       (effects (font (size 1.27 1.27)) (justify left top) hide)
     )
-    (property "Mouser Part Number" "621-DMP21D5UFB4-7B" (at 82.55 -458.09 0)
+    (property "Mouser Part Number" "771-BSS84AKM315" (at 82.55 -458.09 0)
       (effects (font (size 1.27 1.27)) (justify left top) hide)
     )
-    (property "Mouser Price/Stock" "https://www.mouser.co.uk/ProductDetail/Diodes-Incorporated/DMP21D5UFB4-7B?qs=gfe7vQ8txpUVAcG22XiS3g%3D%3D" (at 82.55 -558.09 0)
+    (property "Mouser Price/Stock" "https://www.mouser.co.uk/ProductDetail/Nexperia/BSS84AKM315?qs=A1cBxND5mHI4EQ%2FktSuzZA%3D%3D" (at 82.55 -558.09 0)
       (effects (font (size 1.27 1.27)) (justify left top) hide)
     )

Commit message: PCB V3 progress
Other:
- note added: "PULL OUT Off: 0 X Rx mode: 1 X Tx mode: 1 X"
- note removed: "PULL OUT Off: 0 X Rx mode: 1 0 Tx mode: 1 X"
