File: PCBs/watch_main_v2/display_connector.kicad_sch (KiCad schematic)
At the start: 1 part, among them J702 AXG130144

Commit message: Schematic v2 complete
Connections:
- net +1V8: now also J702.1, J702.2, J702.5
- net DSI.CKN: now also J702.28
- net DSI.CKP: now also J702.27
- net DSI.D0N: now also J702.25
- net DSI.D0P: now also J702.24
- net DSI_TE: now also J702.11
- net ELVDD: now also J702.16, J702.17, J702.18
- net ELVSS: now also J702.13, J702.14, J702.15
- net RESET: now also J702.10
- net SWIRE: now also J702.12
- net TP_RST: now reaches J702.19
- net TP_I2C.SCL: now reaches J702.20
- net TP_I2C.SDA: now reaches J702.21
- net TP_INT: now reaches J702.22
- net GND: now reaches J702.23
- net GND: now also J702.26, J702.29, J702.6, J702.7, J702.8, J702.9
- net AVDD: now reaches J702.3
- net AVDD: now also J702.4
- no-connect marks 0 -> 9
Other:
- moved on the sheet: J702

Commit message: PCB V3 progress
Parts:
- renumbered J702 to J501
