File: PCBs/watch_main_v2/micro_sd.kicad_sch (KiCad schematic)
At the start: 4 parts, among them IC1101 NVT4858HKZ, J1101 105162-0001

Commit message: 190 Unrouted traces
Parts:
- added U1102: NCP45525IMNTWG-H, watch_footprints:NCP45525IMNTWGH, symbol NCP45525IMNTWG-H:NCP45525IMNTWG-H
Connections:
- net +3V3: now also U1102.1 (VIN), U1102.3 (VCC); no longer C1101.1, J1101.4 (VDD)
- net GND: now also U1102.4 (GND), U1102.9 (EP)
- new net +3V3_SD: C1101.1, J1101.4 (VDD), U1102.5 (BLEED), U1102.7 (VOUT_1), U1102.8 (VOUT_2)
- new net EN: U1102.2 (EN)
- no-connect marks 0 -> 1
Other:
- note added: "Active high EN"
- moved on the sheet: C1102, IC1101, J1101
