File: PCBs/watch_main_v2/sensors.kicad_sch (KiCad schematic)
At the start: 10 parts, among them IC1301 IIS2MDCTR, IC1302 OPT3004DNPR, U1301 LSM6DSO16IS

Commit message: Schematic v2 complete
Connections:
- net GND: no longer U1301.1 (SDO/SA0)
- net I2C.SCL: no longer U1301.13 (SCL)
- net I2C.SDA: no longer U1301.14 (SDA)
- net SPI.CS: now reaches U1301.12 (CS)
- new net SPI.MISO: U1301.1 (SDO/SA0)
- new net SPI.MOSI: U1301.14 (SDA)
- new net SPI.SCK: U1301.13 (SCL)
- no-connect marks 8 -> 6
Changed lines of the file:
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@@
   (junction (at 132.08 55.88) (diameter 0) (color 0 0 0 0)
   )
-  (junction (at 111.76 68.58) (diameter 0) (color 0 0 0 0)
-  )
   (junction (at 241.3 58.42) (diameter 0) (color 0 0 0 0)
   )
@@
   )
   (no_connect (at 68.58 124.46))
-  (no_connect (at 68.58 55.88))
   (no_connect (at 68.58 134.62))
   (no_connect (at 68.58 137.16))
-  (no_connect (at 101.6 63.5))
   (no_connect (at 68.58 139.7))
   (no_connect (at 68.58 68.58))
   (no_connect (at 68.58 71.12))
-  (bus_entry (at 53.34 48.26) (size 2.54 2.54)
-    (stroke (width 0) (type default))
-  )
   (bus_entry (at 193.04 45.72) (size 2.54 2.54)
     (stroke (width 0) (type default))
   )
+  (bus_entry (at 50.8 45.72) (size 2.54 2.54)
+    (stroke (width 0) (type default))
+  )
+  (bus_entry (at 50.8 50.8) (size 2.54 2.54)
+    (stroke (width 0) (type default))
+  )
   (bus_entry (at 53.34 116.84) (size 2.54 2.54)
     (stroke (width 0) (type default))
   )
-  (bus_entry (at 53.34 45.72) (size 2.54 2.54)
+  (bus_entry (at 50.8 48.26) (size 2.54 2.54)
+    (stroke (width 0) (type default))
+  )
+  (bus_entry (at 50.8 53.34) (size 2.54 2.54)
     (stroke (width 0) (type default))
   )
@@
     (stroke (width 0) (type default))
   )
-  (wire (pts (xy 55.88 48.26) (xy 68.58 48.26))
-    (stroke (width 0) (type default))
-  )
-  (wire (pts (xy 109.22 63.5) (xy 111.76 63.5))
-    (stroke (width 0) (type default))
-  )
   (wire (pts (xy 111.76 68.58) (xy 109.22 68.58))
     (stroke (width 0) (type default))
@@
     (stroke (width 0) (type default))
   )
+  (bus (pts (xy 50.8 45.72) (xy 50.8 48.26))
+    (stroke (width 0) (type default))
+  )
   (wire (pts (xy 111.76 55.88) (xy 109.22 55.88))
     (stroke (width 0) (type default))
@@
     (stroke (width 0) (type default))
   )
-  (bus (pts (xy 40.64 45.72) (xy 53.34 45.72))
+  (bus (pts (xy 38.1 45.72) (xy 50.8 45.72))
+    (stroke (width 0) (type default))
+  )
+  (wire (pts (xy 50.8 63.5) (xy 68.58 63.5))
+    (stroke (width 0) (type default))
+  )
+  (wire (pts (xy 53.34 53.34) (xy 68.58 53.34))
     (stroke (width 0) (type default))
   )
@@
     (stroke (width 0) (type default))
   )
-  (wire (pts (xy 53.34 60.96) (xy 68.58 60.96))
+  (wire (pts (xy 50.8 60.96) (xy 68.58 60.96))
     (stroke (width 0) (type default))
   )
@@
     (stroke (width 0) (type default))
   )
+  (bus (pts (xy 50.8 50.8) (xy 50.8 53.34))
+    (stroke (width 0) (type default))
+  )
   (wire (pts (xy 111.76 45.72) (xy 111.76 48.26))
     (stroke (width 0) (type default))
   )
+  (wire (pts (xy 53.34 50.8) (xy 68.58 50.8))
+    (stroke (width 0) (type default))
+  )
   (wire (pts (xy 142.24 134.62) (xy 132.08 134.62))
     (stroke (width 0) (type default))
@@
     (stroke (width 0) (type default))
   )
-  (wire (pts (xy 111.76 63.5) (xy 111.76 68.58))
-    (stroke (width 0) (type default))
-  )
   (wire (pts (xy 238.76 60.96) (xy 241.3 60.96))
     (stroke (width 0) (type default))
@@
     (stroke (width 0) (type default))
   )
-  (bus (pts (xy 53.34 45.72) (xy 53.34 48.26))
-    (stroke (width 0) (type default))
-  )
   (wire (pts (xy 142.24 63.5) (xy 142.24 66.04))
     (stroke (width 0) (type default))
@@
     (stroke (width 0) (type default))
   )
+  (wire (pts (xy 53.34 55.88) (xy 68.58 55.88))
+    (stroke (width 0) (type default))
+  )
+  (bus (pts (xy 50.8 48.26) (xy 50.8 50.8))
+    (stroke (width 0) (type default))
+  )
   (wire (pts (xy 142.24 124.46) (xy 132.08 124.46))
     (stroke (width 0) (type default))
@@
     (stroke (width 0) (type default))
   )
-  (wire (pts (xy 53.34 63.5) (xy 68.58 63.5))
-    (stroke (width 0) (type default))
-  )
   (wire (pts (xy 132.08 66.04) (xy 132.08 63.5))
     (stroke (width 0) (type default))
   )
-  (wire (pts (xy 55.88 50.8) (xy 68.58 50.8))
-    (stroke (width 0) (type default))
-  )
   (wire (pts (xy 152.4 134.62) (xy 142.24 134.62))
     (stroke (width 0) (type default))
@@
     (stroke (width 0) (type default))
   )
+  (wire (pts (xy 53.34 48.26) (xy 68.58 48.26))
+    (stroke (width 0) (type default))
+  )
   (text "Address = 0x1E" (at 68.58 154.94 0)
     (effects (font (size 1.27 1.27)) (justify left bottom))
@@
     (effects (font (size 1.27 1.27)) (justify left bottom))
   )
-  (label "IMU_INT2" (at 66.04 63.5 180) (fields_autoplaced)
-    (effects (font (size 1.27 1.27)) (justify right bottom))
+  (label "SPI.SCK" (at 55.88 48.26 0)
+    (effects (font (size 1.27 1.27)) (justify left bottom))
+  )
+  (label "SPI.CS" (at 55.88 55.88 0)
+    (effects (font (size 1.27 1.27)) (justify left bottom))
+  )
+  (label "IMU_INT2" (at 55.88 63.5 0) (fields_autoplaced)
+    (effects (font (size 1.27 1.27)) (justify left bottom))
   )
   (label "ALS_INT" (at 205.74 55.88 180) (fields_autoplaced)
@@
     (effects (font (size 1.27 1.27)) (justify left bottom))
   )
-  (label "I2C.SDA" (at 58.42 50.8 0) (fields_autoplaced)
-    (effects (font (size 1.27 1.27)) (justify left bottom))
-  )
   (label "I2C{I2C}" (at 50.8 114.3 180) (fields_autoplaced)
     (effects (font (size 1.27 1.27)) (justify right bottom))
@@
     (effects (font (size 1.27 1.27)) (justify left bottom))
   )
+  (label "SPI.MISO" (at 55.88 53.34 0)
+    (effects (font (size 1.27 1.27)) (justify left bottom))
+  )
   (label "I2C.SCL" (at 58.42 116.84 0) (fields_autoplaced)
     (effects (font (size 1.27 1.27)) (justify left bottom))
   )
-  (label "IMU_INT1" (at 66.04 60.96 180) (fields_autoplaced)
-    (effects (font (size 1.27 1.27)) (justify right bottom))
-  )
-  (label "I2C.SCL" (at 58.42 48.26 0) (fields_autoplaced)
+  (label "SPI.MOSI" (at 55.88 50.8 0)
+    (effects (font (size 1.27 1.27)) (justify left bottom))
+  )
+  (label "IMU_INT1" (at 55.88 60.96 0) (fields_autoplaced)
     (effects (font (size 1.27 1.27)) (justify left bottom))
   )
@@
     (effects (font (size 1.27 1.27)) (justify left bottom))
   )
-  (label "I2C{I2C}" (at 50.8 45.72 180) (fields_autoplaced)
+  (label "SPI{SPI}" (at 48.26 45.72 180) (fields_autoplaced)
     (effects (font (size 1.27 1.27)) (justify right bottom))
   )
@@
     (effects (font (size 1.27 1.27)) (justify right bottom))
   )
-  (hierarchical_label "IMU_INT1" (shape output) (at 53.34 60.96 180) (fields_autoplaced)
-    (effects (font (size 1.27 1.27)) (justify right))
-  )
-  (hierarchical_label "MAG_INT" (shape output) (at 53.34 129.54 180) (fields_autoplaced)
-    (effects (font (size 1.27 1.27)) (justify right))
-  )
-  (hierarchical_label "ALS_INT" (shape output) (at 193.04 55.88 180) (fields_autoplaced)
-    (effects (font (size 1.27 1.27)) (justify right))
-  )
-  (hierarchical_label "I2C" (shape bidirectional) (at 40.64 45.72 180) (fields_autoplaced)
-    (effects (font (size 1.27 1.27)) (justify right))
-    (property "DSI" "DSI" (at 40.64 46.99 0)
+  (hierarchical_label "IMU_INT1" (shape output) (at 50.8 60.96 180) (fields_autoplaced)
+    (effects (font (size 1.27 1.27)) (justify right))
+  )
+  (hierarchical_label "SPI" (shape bidirectional) (at 38.1 45.72 180) (fields_autoplaced)
+    (effects (font (size 1.27 1.27)) (justify right))
+    (property "DSI" "DSI" (at 38.1 46.99 0)
       (effects (font (size 1.27 1.27) italic) (justify right) hide)
     )
   )
-  (hierarchical_label "IMU_INT2" (shape output) (at 53.34 63.5 180) (fields_autoplaced)
-    (effects (font (size 1.27 1.27)) (justify right))
-  )
+  (hierarchical_label "MAG_INT" (shape output) (at 53.34 129.54 180) (fields_autoplaced)
+    (effects (font (size 1.27 1.27)) (justify right))
+  )
+  (hierarchical_label "ALS_INT" (shape output) (at 193.04 55.88 180) (fields_autoplaced)
+    (effects (font (size 1.27 1.27)) (justify right))
+  )
+  (hierarchical_label "I2C" (shape bidirectional) (at 40.64 114.3 180) (fields_autoplaced)
+    (effects (font (size 1.27 1.27)) (justify right))
+    (property "DSI" "DSI" (at 40.64 115.57 0)
+      (effects (font (size 1.27 1.27) italic) (justify right) hide)
+    )
+  )
+  (hierarchical_label "IMU_INT2" (shape output) (at 50.8 63.5 180) (fields_autoplaced)
+    (effects (font (size 1.27 1.27)) (justify right))
+  )
